File: rgb/pcb/Lily58.kicad_pcb (KiCad board)
At the start: 2 copper layers, 142.5 x 106.3 mm, 117 parts, among them J1 LED, J2 4PIN, P1 i2c_pin, P2 i2c_pin, P3 ICSP, P4 OLED, SW1 SW_PUSH, SW10 SW_PUSH, SW11 SW_PUSH, SW12 SW_PUSH, SW13 SW_PUSH, SW14 SW_PUSH, SW15 SW_PUSH, SW16 SW_PUSH, SW17 SW_PUSH, SW18 SW_PUSH, SW19 SW_PUSH, SW2 SW_PUSH, SW20 SW_PUSH, SW21 SW_PUSH, SW22 SW_PUSH, SW23 SW_PUSH, SW24 SW_PUSH, SW25 SW_PUSH, SW26 SW_PUSH, SW27 SW_PUSH, SW28 SW_PUSH, SW29 SW_PUSH, SW3 SW_PUSH, SW4 SW_PUSH, SW5 SW_PUSH, SW6 SW_PUSH, SW7 SW_PUSH, SW8 SW_PUSH, SW9 SW_PUSH, U1 ProMicro

Commit message: Tighten up some traces
Routing:
- net VCC: track 984.3 -> 975.7 mm, vias 34 -> 33
Changed lines of the file:
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@@
     (pad_to_mask_clearance 0.2)
     (aux_axis_origin 83 37)
-    (visible_elements 7FFFFF7F)
+    (visible_elements 7FFFFFFF)
     (pcbplotparams
       (layerselection 0x010f0_ffffffff)
@@
   (segment (start 180 72.975) (end 180 74.442476) (width 0.5) (layer F.Cu) (net 34))
   (segment (start 141.9 73.075) (end 141.9 74.542476) (width 0.5) (layer F.Cu) (net 34))
-  (segment (start 159.6 74.542476) (end 141.9 74.542476) (width 0.5) (layer F.Cu) (net 34))
-  (segment (start 161 73.142476) (end 159.6 74.542476) (width 0.5) (layer F.Cu) (net 34))
   (segment (start 161 71.675) (end 161 73.142476) (width 0.5) (layer F.Cu) (net 34))
-  (segment (start 182.887486 79.57501) (end 178.877476 75.565) (width 0.5) (layer F.Cu) (net 34))
-  (segment (start 198.68199 79.57501) (end 182.887486 79.57501) (width 0.5) (layer F.Cu) (net 34))
-  (segment (start 199.1 79.157) (end 198.68199 79.57501) (width 0.5) (layer F.Cu) (net 34))
   (segment (start 199.1 77.675) (end 199.1 79.157) (width 0.5) (layer F.Cu) (net 34))
   (segment (start 201.01801 81.07501) (end 199.1 79.157) (width 0.5) (layer F.Cu) (net 34))
@@
   (segment (start 181.745502 71.225) (end 182.233001 71.712499) (width 0.5) (layer B.Cu) (net 34))
   (segment (start 180 71.225) (end 181.745502 71.225) (width 0.5) (layer B.Cu) (net 34))
-  (via (at 159.6 74.542476) (size 0.6) (drill 0.4) (layers F.Cu B.Cu) (net 34))
-  (segment (start 160.242526 74.542476) (end 159.6 74.542476) (width 0.5) (layer B.Cu) (net 34))
-  (segment (start 163.246501 71.538501) (end 160.242526 74.542476) (width 0.5) (layer B.Cu) (net 34))
-  (segment (start 163.246501 70.442499) (end 163.246501 71.538501) (width 0.5) (layer B.Cu) (net 34))
-  (segment (start 162.729002 69.925) (end 163.246501 70.442499) (width 0.5) (layer B.Cu) (net 34))
-  (segment (start 161 69.925) (end 162.729002 69.925) (width 0.5) (layer B.Cu) (net 34))
   (via (at 141.9 74.542476) (size 0.6) (drill 0.4) (layers F.Cu B.Cu) (net 34))
   (segment (start 142.542526 74.542476) (end 141.9 74.542476) (width 0.5) (layer B.Cu) (net 34))
@@
   (segment (start 141.9 74.542476) (end 141.467466 74.97501) (width 0.5) (layer F.Cu) (net 34))
   (segment (start 141.467466 74.97501) (end 134.667964 74.97501) (width 0.5) (layer F.Cu) (net 34))
-  (segment (start 159.899999 74.842475) (end 159.6 74.542476) (width 0.5) (layer F.Cu) (net 34))
-  (segment (start 159.994544 74.93702) (end 159.899999 74.842475) (width 0.5) (layer F.Cu) (net 34))
-  (segment (start 178.249496 74.93702) (end 159.994544 74.93702) (width 0.5) (layer F.Cu) (net 34))
   (segment (start 178.877476 75.565) (end 178.249496 74.93702) (width 0.5) (layer F.Cu) (net 34))
   (segment (start 137.1 51.225) (end 136.4845 50.6095) (width 0.5) (layer F.Cu) (net 34))
@@
   (segment (start 126.873 110.2995) (end 126.873 112.776) (width 0.5) (layer B.Cu) (net 34))
   (segment (start 126.873 112.776) (end 125.174 114.475) (width 0.5) (layer B.Cu) (net 34))
+  (segment (start 198.68199 79.57501) (end 199.1 79.157) (width 0.5) (layer F.Cu) (net 34))
+  (segment (start 185.327138 79.57501) (end 198.68199 79.57501) (width 0.5) (layer F.Cu) (net 34))
+  (segment (start 181.317128 75.565) (end 185.327138 79.57501) (width 0.5) (layer F.Cu) (net 34))
+  (segment (start 178.877476 75.565) (end 181.317128 75.565) (width 0.5) (layer F.Cu) (net 34))
+  (segment (start 164.797604 73.142476) (end 161 73.142476) (width 0.5) (layer F.Cu) (net 34))
+  (segment (start 166.592148 74.93702) (end 164.797604 73.142476) (width 0.5) (layer F.Cu) (net 34))
+  (segment (start 168.07748 74.93702) (end 166.592148 74.93702) (width 0.5) (layer F.Cu) (net 34))
+  (segment (start 178.249496 74.93702) (end 168.07748 74.93702) (width 0.5) (layer F.Cu) (net 34))
+  (segment (start 160.567466 73.57501) (end 161 73.142476) (width 0.5) (layer F.Cu) (net 34))
+  (segment (start 156.48549 73.57501) (end 160.567466 73.57501) (width 0.5) (layer F.Cu) (net 34))
+  (segment (start 155.68499 72.77451) (end 156.48549 73.57501) (width 0.5) (layer F.Cu) (net 34))
+  (segment (start 147.31649 72.77451) (end 155.68499 72.77451) (width 0.5) (layer F.Cu) (net 34))
+  (segment (start 145.548524 74.542476) (end 147.31649 72.77451) (width 0.5) (layer F.Cu) (net 34))
+  (segment (start 141.9 74.542476) (end 145.548524 74.542476) (width 0.5) (layer F.Cu) (net 34))
   (segment (start 84.15 45.6) (end 90.1 45.6) (width 0.5) (layer F.Cu) (net 35))
   (segment (start 93.25763 48.75) (end 93.389884 48.617746) (width 0.5) (layer F.Cu) (net 35))
