File: pcb/Lily58.kicad_pcb (KiCad board)
At the start: 2 copper layers, 142.5 x 106.3 mm, 88 parts, among them J1 LED, J2 4PIN, P1 i2c_pin, P2 i2c_pin, P3 ICSP, SW1 SW_PUSH, SW10 SW_PUSH, SW11 SW_PUSH, SW12 SW_PUSH, SW13 SW_PUSH, SW14 SW_PUSH, SW15 SW_PUSH, SW16 SW_PUSH, SW17 SW_PUSH, SW18 SW_PUSH, SW19 SW_PUSH, SW2 SW_PUSH, SW20 SW_PUSH, SW21 SW_PUSH, SW22 SW_PUSH, SW23 SW_PUSH, SW24 SW_PUSH, SW25 SW_PUSH, SW26 SW_PUSH, SW27 SW_PUSH, SW28 SW_PUSH, SW29 SW_PUSH, SW3 SW_PUSH, SW4 SW_PUSH, SW5 SW_PUSH, SW6 SW_PUSH, SW7 SW_PUSH, SW8 SW_PUSH, SW9 SW_PUSH, U1 ProMicro

Commit message: Move files to root directory
Parts:
- added L1: SK6812mini, Lily58-footprint:SK6812MINI_rev, F.Cu at (120.5, 55.5)
- added L10: SK6812mini, Lily58-footprint:SK6812MINI_rev, F.Cu at (177.6, 72.1)
- added L11: SK6812mini, Lily58-footprint:SK6812MINI_rev, F.Cu at (196.7, 76.8)
- added L12: SK6812mini, Lily58-footprint:SK6812MINI_rev, F.Cu at (215.7, 78.3)
- added L13: SK6812mini, Lily58-footprint:SK6812MINI_rev, F.Cu at (120.5, 93.6)
- added L14: SK6812mini, Lily58-footprint:SK6812MINI_rev, F.Cu at (139.5, 91.2)
- added L15: SK6812mini, Lily58-footprint:SK6812MINI_rev, F.Cu at (158.6, 89.9)
- added L16: SK6812mini, Lily58-footprint:SK6812MINI_rev, F.Cu at (177.6, 91.2)
- added L17: SK6812mini, Lily58-footprint:SK6812MINI_rev, F.Cu at (196.7, 96.0)
- added L18: SK6812mini, Lily58-footprint:SK6812MINI_rev, F.Cu at (215.7, 97.5)
- added L19: SK6812mini, Lily58-footprint:SK6812MINI_rev, F.Cu at (120.5, 112.6)
- added L2: SK6812mini, Lily58-footprint:SK6812MINI_rev, F.Cu at (139.5, 53.1)
- added L20: SK6812mini, Lily58-footprint:SK6812MINI_rev, F.Cu at (139.5, 110.3)
- added L21: SK6812mini, Lily58-footprint:SK6812MINI_rev, F.Cu at (158.6, 108.9)
- added L22: SK6812mini, Lily58-footprint:SK6812MINI_rev, F.Cu at (177.6, 110.3)
- added L23: SK6812mini, Lily58-footprint:SK6812MINI_rev, F.Cu at (196.7, 115.0)
- added L24: SK6812mini, Lily58-footprint:SK6812MINI_rev, F.Cu at (215.8, 116.5)
- added L25: SK6812mini, Lily58-footprint:SK6812MINI_rev, F.Cu at (101.4, 103.0)
- added L26: SK6812mini, Lily58-footprint:SK6812MINI_rev, F.Cu at (100.2, 129.8)
- added L27: SK6812mini, Lily58-footprint:SK6812MINI_rev, F.Cu at (130.0, 131.5)
- added L28: SK6812mini, Lily58-footprint:SK6812MINI_rev, F.Cu at (149.0, 129.2)
- added L29: SK6812mini, Lily58-footprint:SK6812MINI_rev, F.Cu at (168.1, 129.2)
- added L3: SK6812mini, Lily58-footprint:SK6812MINI_rev, F.Cu at (158.6, 51.7)
- added L30: SK6812mini, Lily58-footprint:SK6812MINI_underglow_rev, F.Cu at (120.5, 60.2)
- added L31: SK6812mini, Lily58-footprint:SK6812MINI_underglow_rev, F.Cu at (158.6, 56.5)
- added L32: SK6812mini, Lily58-footprint:SK6812MINI_underglow_rev, F.Cu at (196.7, 62.6)
- added L33: SK6812mini, Lily58-footprint:SK6812MINI_underglow_rev, F.Cu at (120.5, 117.3)
- added L34: SK6812mini, Lily58-footprint:SK6812MINI_underglow_rev, F.Cu at (158.6, 113.7)
- added L35: SK6812mini, Lily58-footprint:SK6812MINI_underglow_rev, F.Cu at (196.7, 100.8)
- added L4: SK6812mini, Lily58-footprint:SK6812MINI_rev, F.Cu at (177.6, 53.1)
- added L5: SK6812mini, Lily58-footprint:SK6812MINI_rev, F.Cu at (196.7, 57.9)
- added L6: SK6812mini, Lily58-footprint:SK6812MINI_rev, F.Cu at (215.7, 59.4)
- added L7: SK6812mini, Lily58-footprint:SK6812MINI_rev, F.Cu at (120.5, 74.6)
- added L8: SK6812mini, Lily58-footprint:SK6812MINI_rev, F.Cu at (139.5, 72.2)
- added L9: SK6812mini, Lily58-footprint:SK6812MINI_rev, F.Cu at (158.6, 70.8)
- D1, D10, D11, D12, D13, D14, D15, D16, D17, D18, D19, D2, D20, D21, D22, D23, D24, D25, D27, D28, D29, D3, D4, D5, D6, D7, D8, D9: moved to B.Cu
- JP1, JP2, JP3, JP4, JP5, JP6, JP7, JP8: value (none) -> Jumper_NO_Small
- SW1, SW10, SW11, SW12, SW13, SW14, SW15, SW16, SW17, SW18, SW19, SW2, SW20, SW21, SW22, SW23, SW24, SW25, SW27, SW28, SW29, SW3, SW4, SW5, SW6, SW7, SW8, SW9: footprint Lily58-footprint:MX_PG1350-Under_FLIP_HOLES_18mm -> Lily58-footprint:MX_PG1350_FLIP_HOLES_18mm
- SW26: footprint Lily58-footprint:MX_PG1350-Under_FLIP_HOLES_27mm -> Lily58-footprint:MX_PG1350_FLIP_HOLES_27mm
- TH1, TH2: footprint Lily58-footprint:M2_HOLE_PCB -> Lily58-footprint:HOLE_M2
- moved D12 1.71 mm to (206.2, 73.0), turned to 90 degrees
- moved D24 1.63 mm to (206.2, 111.1), turned to 90 degrees
- turned D1 to 90 degrees
- turned D10 to 90 degrees
- turned D11 to 90 degrees
- turned D13 to 90 degrees
- turned D14 to 90 degrees
- turned D15 to 90 degrees
- turned D16 to 90 degrees
- turned D17 to 90 degrees
- turned D18 to 90 degrees
- turned D19 to 90 degrees
- turned D2 to 90 degrees
- turned D20 to 90 degrees
- turned D21 to 90 degrees
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- renumbered OLED to P4
Routing:
- net GND: track 117.4 -> 1068.1 mm, vias 4 -> 74
- net VCC: track 94.8 -> 1030.4 mm, vias 3 -> 43
- net col1: track 245.7 -> 382.1 mm
- net col4: track 204.8 -> 291.3 mm
- net col5: track 135.9 -> 215.5 mm, vias 0 -> 2
- net col3: track 229.7 -> 300.9 mm
- net col2: track 246.8 -> 314.4 mm
- net Net-(L26-Pad1): track 0.00 -> 64.0 mm, vias 0 -> 3
- net LED: track 63.8 -> 121.3 mm, vias 2 -> 5
- net Net-(L34-Pad1): track 0.00 -> 53.6 mm, vias 0 -> 4
- net col0: track 217.9 -> 270.9 mm
- net Net-(L25-Pad1): track 0.00 -> 52.5 mm, vias 0 -> 2
- net Net-(L32-Pad3): track 0.00 -> 49.9 mm, vias 0 -> 3
- net Net-(L31-Pad3): track 0.00 -> 45.2 mm, vias 0 -> 3
- net Net-(L30-Pad3): track 0.00 -> 44.6 mm, vias 0 -> 3
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Other:
- outline, holes or cut-outs redrawn
- board text added: "Glow"
- board text added: "Lily58 × qtkb"
- board text removed: "PCB Design by F_YUUCHI"
