File: pcb/Lily58.sch (KiCad schematic (older format))
At the start: 84 parts, among them J1 LED, J2 4PIN, P1 i2c_pin, P2 i2c_pin, P3 ICSP, P4 OLED, SW1 SW_PUSH, SW10 SW_PUSH, SW11 SW_PUSH, SW12 SW_PUSH, SW13 SW_PUSH, SW14 SW_PUSH, SW15 SW_PUSH, SW16 SW_PUSH, SW17 SW_PUSH, SW18 SW_PUSH, SW19 SW_PUSH, SW2 SW_PUSH, SW20 SW_PUSH, SW21 SW_PUSH, SW22 SW_PUSH, SW23 SW_PUSH, SW24 SW_PUSH, SW25 SW_PUSH, SW26 SW_PUSH, SW27 SW_PUSH, SW28 SW_PUSH, SW29 SW_PUSH, SW3 SW_PUSH, SW4 SW_PUSH, SW5 SW_PUSH, SW6 SW_PUSH, SW7 SW_PUSH, SW8 SW_PUSH, SW9 SW_PUSH, U1 ProMicro

Commit message: Move files to root directory
Parts:
- added L1, L10, L11, L12, L13, L14, L15, L16, L17, L18, L19, L2, L20, L21, L22, L23, L24, L25, L26, L27, L28, L29, L3, L4, L5, L6, L7, L8, L9: SK6812mini, Lily58-footprint:SK6812MINI_rev, symbol LED:SK6812MINI
- added L30, L31, L32, L33, L34, L35: SK6812mini, Lily58-footprint:SK6812MINI_underglow_rev, symbol LED:SK6812MINI
- D1, D10, D11, D12, D13, D14, D15, D16, D17, D18, D19, D2, D20, D21, D22, D23, D24, D25, D26, D27, D28, D29, D3, D4, D5, D6, D7, D8, D9: symbol Lily58-cache:D -> Lily58-rescue:D-Lily58-cache
- J1: symbol Lily58-cache:LED -> Lily58-rescue:LED-Lily58-cache
- J2: symbol Lily58-cache:MJ-4PP-9 -> Lily58-rescue:MJ-4PP-9-Lily58-cache
- P1, P2: symbol Lily58-cache:i2c_pin -> Lily58-rescue:i2c_pin-Lily58-cache
- P3: symbol Lily58-cache:CONN_01X06 -> Lily58-rescue:CONN_01X06-Lily58-cache
- P4: symbol Lily58-cache:CONN_01X04 -> Lily58-rescue:CONN_01X04-Lily58-cache
- R1, R2: symbol Lily58-cache:R -> Lily58-rescue:R-Lily58-cache
- RSW1: symbol Lily58-cache:SW_RST -> Lily58-rescue:SW_RST-Lily58-cache
- SW1, SW10, SW11, SW12, SW13, SW14, SW15, SW16, SW17, SW18, SW19, SW2, SW20, SW21, SW22, SW23, SW24, SW25, SW27, SW28, SW29, SW3, SW4, SW5, SW6, SW7, SW8, SW9: footprint Lily58-footprint:MX_PG1350-Under_FLIP_HOLES_18mm -> Lily58-footprint:MX_PG1350_FLIP_HOLES_18mm; symbol Lily58-cache:SW_PUSH -> Lily58-rescue:SW_PUSH-Lily58-cache
- SW26: footprint Lily58-footprint:MX_PG1350-Under_FLIP_HOLES_27mm -> Lily58-footprint:MX_PG1350_FLIP_HOLES_27mm; symbol Lily58-cache:SW_PUSH -> Lily58-rescue:SW_PUSH-Lily58-cache
- TH1, TH2, TH3, TH4, TH5, TH6, TH7: symbol Lily58-cache:HOLE -> Lily58-rescue:HOLE-Lily58-cache
- U1: symbol Lily58-cache:ProMicro_2 -> Lily58-rescue:ProMicro_2-Lily58-cache
Connections:
- wire segments 84 -> 200
- no-connect marks 4 -> 5
