File: PCB/MX/FR4_Top_Plate.kicad_pcb (KiCad board)
At the start: 2 copper layers, 139.1 x 106.7 mm, 35 parts, among them SW1 SW_PUSH, SW10 SW_PUSH, SW11 SW_PUSH, SW12 SW_PUSH, SW13 SW_PUSH, SW14 SW_PUSH, SW15 SW_PUSH, SW16 SW_PUSH, SW18 SW_PUSH, SW19 SW_PUSH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

Commit message: added gerbers MX version
Routing:
- added copper zone on B.Cu, net (none)
- added copper zone on F.Cu, net (none)
- removed copper zone on B.Cu, net GND
- removed copper zone on F.Cu, net GND
