File: PCB/Glow/Choc/Lotus58_Glow_Choc.kicad_pcb (KiCad board)
At the start: 2 copper layers, 139.1 x 106.7 mm, 121 parts, among them J1 AudioJack4, P4 OLED, SW1 SW_PUSH, SW10 SW_PUSH, SW11 SW_PUSH, SW12 SW_PUSH, SW13 SW_PUSH, SW14 SW_PUSH, SW15 SW_PUSH, SW16 SW_PUSH, SW17 SW_PUSH, SW18 SW_PUSH, SW19 SW_PUSH, SW2 SW_PUSH, SW20 SW_PUSH, SW21 SW_PUSH, SW22 SW_PUSH, SW23 SW_PUSH, SW24 SW_PUSH, SW25 SW_PUSH, SW26 SW_PUSH, SW27 SW_PUSH, SW28 SW_PUSH, SW29 SW_PUSH, SW3 SW_PUSH, SW30 Rotary_Encoder_Switch, SW4 SW_PUSH, SW5 SW_PUSH, SW6 SW_PUSH, SW7 SW_PUSH, SW8 SW_PUSH, SW9 SW_PUSH, U1 ProMicro

Commit message: Revised footprint
Parts:
- SW1, SW10, SW11, SW12, SW13, SW14, SW15, SW16, SW17, SW18, SW19, SW2, SW20, SW21, SW22, SW23, SW24, SW25, SW26, SW27, SW28, SW29, SW3, SW4, SW5, SW6, SW7, SW8, SW9: footprint keyswitches:Kailh_socket_PG1350_reversible -> keyswitches:Kailh_socket_PG1350_PG1353_reversible
- moved L2 10.0 mm to (133.4, 42.6)
- moved L1 10.0 mm to (114.4, 45.0)
- moved L10 10.0 mm to (171.6, 61.7)
- moved L11 10.0 mm to (190.6, 66.5)
- moved L12 10.0 mm to (209.7, 68.0)
- moved L13 10.0 mm to (114.4, 83.2)
- moved L14 10.0 mm to (133.4, 80.8)
- moved L15 10.0 mm to (152.5, 79.4)
- moved L16 10.0 mm to (171.6, 80.8)
- moved L3 10.0 mm to (152.5, 41.3)
- moved L4 10.0 mm to (171.6, 42.6)
- moved L7 10.0 mm to (114.4, 64.1)
- moved L8 10.0 mm to (133.4, 61.7)
- moved L9 10.0 mm to (152.5, 60.3)
- moved L5 10.0 mm to (190.6, 47.5)
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Routing:
- net VCC: track 874.7 -> 311.6 mm, vias 40 -> 13
- net col5: track 212.7 -> 23.4 mm, vias 11 -> 1
- net col3: track 283.4 -> 94.9 mm, vias 12 -> 3
- net col1: track 310.7 -> 148.3 mm, vias 13 -> 6
- net col2: track 299.1 -> 145.4 mm, vias 12 -> 5
- net col4: track 279.7 -> 150.8 mm, vias 13 -> 7
- net row3: track 184.0 -> 91.8 mm
- net col0: track 309.8 -> 236.4 mm, vias 11 -> 7
- net row1: track 148.0 -> 78.7 mm
- net Net-(L29-Pad1): track 53.6 -> 4.83 mm, vias 2 -> 1
- net Net-(L13-Pad3): track 33.5 -> 0.00 mm, vias 2 -> 0
- net Net-(L18-Pad1): track 33.1 -> 0.00 mm, vias 2 -> 0
- net Net-(L12-Pad3): track 32.7 -> 0.00 mm, vias 2 -> 0
- net Net-(L26-Pad1): track 32.4 -> 0.43 mm, vias 2 -> 0
- net Net-(L19-Pad1): track 27.8 -> 0.45 mm, vias 2 -> 0
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