File: PCB/Glow/MX/Lotus58_Glow.kicad_pcb (KiCad board)
At the start: 2 copper layers, 139.1 x 106.7 mm, 121 parts, among them J1 AudioJack4, P4 OLED, SW1 SW_PUSH, SW10 SW_PUSH, SW11 SW_PUSH, SW12 SW_PUSH, SW13 SW_PUSH, SW14 SW_PUSH, SW15 SW_PUSH, SW16 SW_PUSH, SW17 SW_PUSH, SW18 SW_PUSH, SW19 SW_PUSH, SW2 SW_PUSH, SW20 SW_PUSH, SW21 SW_PUSH, SW22 SW_PUSH, SW23 SW_PUSH, SW24 SW_PUSH, SW25 SW_PUSH, SW26 SW_PUSH, SW27 SW_PUSH, SW28 SW_PUSH, SW29 SW_PUSH, SW3 SW_PUSH, SW30 Rotary_Encoder_Switch, SW4 SW_PUSH, SW5 SW_PUSH, SW6 SW_PUSH, SW7 SW_PUSH, SW8 SW_PUSH, SW9 SW_PUSH, U1 ProMicro

Commit message: Added optional encoder layout
Parts:
- added SW31: Rotary_Encoder_Switch, Keebio-Parts:RotaryEncoder_EC11-no-legs, F.Cu at (90.5, 98.3)
- moved D25 11.6 mm to (100.1, 98.3), turned to 90 degrees
- moved L25 0.56 mm to (90.5, 102.8)
Connections:
- net Enc0 renamed B
- net Enc1 renamed A
- net Net-(D25-Pad2) renamed Alt
Routing:
- net B: track 40.7 -> 109.8 mm, vias 2 -> 5
- net A: track 39.1 -> 99.4 mm, vias 1 -> 5
- net col5: track 212.7 -> 221.9 mm
- net Alt: track 15.6 -> 22.9 mm
- net row4: track 145.3 -> 141.3 mm
- net Net-(L25-Pad1): track 31.9 -> 33.6 mm
- net VCC: track 874.7 -> 875.9 mm
- net Net-(L19-Pad1): track 27.8 -> 28.5 mm

Commit message: Updated silkscreen
New name!
Other:
- board text added: "Lotus 58 Glow"
- board text added: "Markus Knutsson 2020"
- board text added: "https://github.com/TweetyDaBird"
- board text removed: "Markus Knutsson 2020 https://github.com/TweetyDaBird"
- board text removed: "Split 58 HS-RGB"

Commit message: Revised footprint
Parts:
- L2, L30: moved to B.Cu
- SW1, SW10, SW11, SW12, SW13, SW14, SW15, SW16, SW17, SW18, SW19, SW2, SW20, SW21, SW22, SW23, SW24, SW25, SW27, SW28, SW29, SW3, SW4, SW5, SW6, SW7, SW8, SW9: footprint Keyboard Library:Cherry_MX_Kaihl_HS_1.0u_Reversible -> keyswitches:Kailh_socket_MX_reversible_RGB
- SW26: footprint Keyboard Library:Cherry_MX_Kaihl_HS_1.5u_Reversible -> keyswitches:Kailh_socket_MX_reversible_RGB
- moved L30 16.6 mm to (200.0, 112.5)
- moved JP12 15.6 mm to (99.9, 71.6)
- moved JP13 15.6 mm to (99.9, 71.6)
- moved C2 15.0 mm to (104.4, 55.9), turned to 135 degrees
- moved C1 14.7 mm to (104.8, 53.3), turned to 315 degrees
- moved L31 14.7 mm to (152.4, 128.1), turned to 180 degrees
- moved D25 13.8 mm to (90.7, 88.3), turned to 180 degrees
- moved D20 13.6 mm to (133.7, 95.7), turned to 180 degrees
- moved D3 13.5 mm to (152.5, 37.2), turned to 180 degrees
- moved D9 13.3 mm to (152.5, 56.2), turned to 180 degrees
- moved D8 13.1 mm to (133.4, 57.6), turned to 180 degrees
- moved D12 13.1 mm to (209.6, 63.9), turned to 180 degrees
- moved D14 12.9 mm to (133.4, 76.6), turned to 180 degrees
- moved D29 12.9 mm to (161.9, 114.7), turned to 180 degrees
- moved D21 12.9 mm to (152.5, 94.3), turned to 180 degrees
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Connections:
- L2 pad 3: Net-(L1-Pad1) -> Net-(L2-Pad3)
- L24 pad 1: Net-(L23-Pad3) -> Net-(L24-Pad1)
- L25 pad 3: Net-(L19-Pad1) -> Net-(L25-Pad3)
- L29 pad 3: Net-(L28-Pad1) -> Net-(L29-Pad3)
- L30 pad 1: Net-(L30-Pad1) -> Net-(L23-Pad3)
- L30 pad 3: Net-(L29-Pad1) -> Net-(L24-Pad1)
- L31 pad 1: Net-(L31-Pad1) -> Net-(L29-Pad3)
- L31 pad 3: Net-(L30-Pad1) -> Net-(L28-Pad1)
- L32 pad 1: Net-(L32-Pad1) -> Net-(L25-Pad3)
- L32 pad 3: Net-(L31-Pad1) -> Net-(L19-Pad1)
- L34 pad 1: Net-(L33-Pad3) -> Net-(L34-Pad1)
- L34 pad 3: Net-(L34-Pad3) -> Net-(L3-Pad1)
- L35 pad 1: Net-(L34-Pad3) -> Net-(L2-Pad3)
- L35 pad 3: Net-(L32-Pad1) -> Net-(L1-Pad1)
- L4 pad 3: Net-(L3-Pad1) -> Net-(L34-Pad1)
- L5 pad 1: Net-(L5-Pad1) -> Net-(L33-Pad3)
- L6 pad 3: Net-(L5-Pad1) -> Net-(L33-Pad1)
- SW31 pad S1: Alt -> col5
- SW31 pad S2: col5 -> Alt
- U1 pad 10: row2 -> row3
- U1 pad 11: row3 -> row4
- U1 pad 12: row4 -> Hand
- U1 pad 13: col0 -> col3
- U1 pad 16: col3 -> col0
- U1 pad 7: Hand -> row0
- U1 pad 8: row0 -> row1
- U1 pad 9: row1 -> row2
Routing:
- net col0: track 309.8 -> 203.0 mm, vias 11 -> 6
- net col4: track 279.7 -> 183.7 mm, vias 13 -> 9
- net col3: track 283.4 -> 200.0 mm, vias 12 -> 10
- net col2: track 299.1 -> 219.3 mm, vias 12 -> 10
- net Net-(L32-Pad1): track 76.7 -> 0.00 mm, vias 2 -> 0
- net col5: track 221.9 -> 155.9 mm, vias 11 -> 8
- net col1: track 310.7 -> 246.9 mm, vias 13 -> 8
- net Net-(L30-Pad1): track 54.9 -> 0.00 mm, vias 4 -> 0
- net Net-(L29-Pad1): track 53.6 -> 3.49 mm, vias 2 -> 1
- net Net-(L34-Pad3): track 44.8 -> 0.00 mm, vias 2 -> 0
- net Net-(L31-Pad1): track 44.5 -> 0.00 mm, vias 2 -> 0
- net VCC: track 875.9 -> 843.3 mm, vias 40 -> 45
- net GND: track 64.1 -> 35.3 mm, vias 65 -> 45
- net Net-(L33-Pad3): track 35.2 -> 10.6 mm
- net Net-(L5-Pad1): track 20.7 -> 0.00 mm, vias 2 -> 0
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Other:
- board size 139.1 x 106.7 mm -> 139.1 x 107.7 mm

Commit message: Updated Plates
Parts:
- renumbered RESET1 to RESET
Routing:
- net col1: track 246.9 -> 245.5 mm, vias 8 -> 12
- net B: track 90.2 -> 90.9 mm
- net Net-(D26-Pad2): vias 1 -> 2
- net Net-(D3-Pad2): vias 1 -> 2
- net col5: vias 8 -> 12
- net col4: vias 9 -> 13
- net col3: vias 10 -> 14
- net col2: vias 10 -> 14
- net col0: vias 6 -> 9
- net Net-(D9-Pad2): vias 1 -> 2
- net Net-(D8-Pad2): vias 1 -> 2
- net Net-(D7-Pad2): vias 1 -> 2
- net Net-(D6-Pad2): vias 1 -> 2
- net Net-(D5-Pad2): vias 1 -> 2
- net Net-(D4-Pad2): vias 1 -> 2
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