File: PCB/Glow/MX/Lotus58_Glow.sch (KiCad schematic (older format))
At the start: 122 parts, among them J1 AudioJack4, P4 OLED, SW1 SW_PUSH, SW10 SW_PUSH, SW11 SW_PUSH, SW12 SW_PUSH, SW13 SW_PUSH, SW14 SW_PUSH, SW15 SW_PUSH, SW16 SW_PUSH, SW17 SW_PUSH, SW18 SW_PUSH, SW19 SW_PUSH, SW2 SW_PUSH, SW20 SW_PUSH, SW21 SW_PUSH, SW22 SW_PUSH, SW23 SW_PUSH, SW24 SW_PUSH, SW25 SW_PUSH, SW26 SW_PUSH, SW27 SW_PUSH, SW28 SW_PUSH, SW29 SW_PUSH, SW3 SW_PUSH, SW30 Rotary_Encoder_Switch, SW31 Rotary_Encoder_Switch, SW4 SW_PUSH, SW5 SW_PUSH, SW6 SW_PUSH, SW7 SW_PUSH, SW8 SW_PUSH, SW9 SW_PUSH, U1 ProMicro

Commit message: Revised footprint
Parts:
- SW1, SW10, SW11, SW12, SW13, SW14, SW15, SW16, SW17, SW18, SW19, SW2, SW20, SW21, SW22, SW23, SW24, SW25, SW27, SW28, SW29, SW3, SW4, SW5, SW6, SW7, SW8, SW9: footprint Keyboard Library:Cherry_MX_Kaihl_HS_1.0u_Reversible -> keyswitches:Kailh_socket_MX_reversible_RGB
- SW26: footprint Keyboard Library:Cherry_MX_Kaihl_HS_1.5u_Reversible -> keyswitches:Kailh_socket_MX_reversible_RGB
Connections:
- net Alt: now also SW31.S2; no longer SW31.S1
- net Hand: now also U1.12 (9/PB5); no longer U1.7 (4/PD4)
- net col0: now also U1.16 (15/PB1/SCLK); no longer U1.13 (10/PB6)
- net col3: now also U1.13 (10/PB6); no longer U1.16 (15/PB1/SCLK)
- net col5: now also SW31.S1; no longer SW31.S2
- net row0: now also U1.7 (4/PD4); no longer U1.8 (5/PC6)
- net row1: now also U1.8 (5/PC6); no longer U1.9 (6/PD7)
- net row2: now also U1.9 (6/PD7); no longer U1.10 (7/PE6)
- net row3: now also U1.10 (7/PE6); no longer U1.11 (8/PB4)
- net row4: now also U1.11 (8/PB4); no longer U1.12 (9/PB5)
- net at L1.1 (DOUT): now also L35.3 (DIN); no longer L2.3 (DIN)
- net at L3.1 (DOUT): now also L34.3 (DIN); no longer L4.3 (DIN)
- net at L5.1 (DOUT): now also L33.3 (DIN); no longer L6.3 (DIN)
- net at L19.1 (DOUT): now also L32.3 (DIN); no longer L25.3 (DIN)
- net at L23.3 (DIN): now also L30.1 (DOUT); no longer L24.1 (DOUT)
- net at L28.1 (DOUT): now also L31.3 (DIN); no longer L29.3 (DIN)
- net at L30.3 (DIN): now also L24.1 (DOUT); no longer L29.1 (DOUT)
- net at L31.1 (DOUT): now also L29.3 (DIN); no longer L32.3 (DIN)
- net at L32.1 (DOUT): now also L25.3 (DIN); no longer L35.3 (DIN)
- net at L35.1 (DOUT): now also L2.3 (DIN); no longer L34.3 (DIN)
- net at L34.1 (DOUT): now also L4.3 (DIN); no longer L33.3 (DIN)
- net at L33.1 (DOUT): now also L6.3 (DIN)
Other:
- moved on the sheet: L1, L10, L11, L12, L13, L14, L15, L16, L17, L18, L19, L2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

Commit message: Adjusted plate
Other:
- moved on the sheet: J1, JP10, JP11, JP9
