File: Plate/Glow/MX/FR4_Bottom_Plate.kicad_pcb (KiCad board)
At the start: 2 copper layers, 139.1 x 106.7 mm, 5 parts

Commit message: Updated Plates
Other:
- board size 139.1 x 106.7 mm -> 139.1 x 107.7 mm
- board text removed: "Split 58 HS-RGB"
Changed lines of the file:
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@@
   (general
     (thickness 1.6)
-    (drawings 64)
+    (drawings 62)
     (tracks 0)
     (zones 0)
@@
   (page A4)
   (title_block
-    (title "(Not!)Lily58")
-    (date 2020-11-12)
-    (rev 0.9)
+    (title "Lotus 58 Glow MX")
+    (date 2020-12-12)
+    (rev 0.95)
     (company "Markus Knutsson <markus.knutsson@tweety.se>")
     (comment 1 https://github.com/TweetyDaBird)
@@
     (uvia_drill 0.1)
   )
-  (module MountingHole:MountingHole_2.7mm_M2.5 (layer F.Cu)
+  (module MountingHole:MountingHole_2.7mm_M2.5 locked (layer F.Cu)
     (at 98.8949 114.1095 90)
     (descr "Mounting Hole 2.7mm, no annular, M2.5")
@@
     (pad 1 np_thru_hole circle (at 0 0 90) (size 2.7 2.7) (drill 2.7) (layers *.Cu *.Mask))
   )
-  (module MountingHole:MountingHole_2.7mm_M2.5 (layer F.Cu)
+  (module MountingHole:MountingHole_2.7mm_M2.5 locked (layer F.Cu)
     (at 199.7 100)
     (descr "Mounting Hole 2.7mm, no annular, M2.5")
@@
     (pad 1 np_thru_hole circle (at 0 0) (size 2.7 2.7) (drill 2.7) (layers *.Cu *.Mask))
   )
-  (module MountingHole:MountingHole_2.7mm_M2.5 (layer F.Cu)
+  (module MountingHole:MountingHole_2.7mm_M2.5 locked (layer F.Cu)
     (at 124.3965 95.5675)
     (descr "Mounting Hole 2.7mm, no annular, M2.5")
@@
     (pad 1 np_thru_hole circle (at 0 0) (size 2.7 2.7) (drill 2.7) (layers *.Cu *.Mask))
   )
-  (module MountingHole:MountingHole_2.7mm_M2.5 (layer F.Cu)
+  (module MountingHole:MountingHole_2.7mm_M2.5 locked (layer F.Cu)
     (at 199.7 61.8)
     (descr "Mounting Hole 2.7mm, no annular, M2.5")
@@
     (pad 1 np_thru_hole circle (at 0 0) (size 2.7 2.7) (drill 2.7) (layers *.Cu *.Mask))
   )
-  (module MountingHole:MountingHole_2.7mm_M2.5 (layer F.Cu)
+  (module MountingHole:MountingHole_2.7mm_M2.5 locked (layer F.Cu)
     (at 124.32538 57.40908)
     (descr "Mounting Hole 2.7mm, no annular, M2.5")
@@
     (arrow2a (pts (xy 219.70492 21.844) (xy 218.578416 21.257579)))
     (arrow2b (pts (xy 219.70492 21.844) (xy 218.578416 22.430421)))
-  )
-  (gr_text "Split 58 HS-RGB" (at 92.0115 109.855) (layer B.SilkS)
-    (effects (font (size 1.5 1.5) (thickness 0.3)) (justify mirror))
-  )
-  (gr_text "Split 58 HS-RGB" (at 92.0115 109.855) (layer F.SilkS)
-    (effects (font (size 1.5 1.5) (thickness 0.3)))
   )
   (gr_line (start 80.7085 111.8235) (end 80.772 112.649) (layer Edge.Cuts) (width 0.2))
@@
   (gr_line (start 172.290391 123.987771) (end 172.494174 123.330573) (layer Edge.Cuts) (width 0.2))
   (gr_line (start 172.19422 124.69622) (end 172.290391 123.987771) (layer Edge.Cuts) (width 0.2))
-  (gr_line (start 217.79552 42.621355) (end 181.0004 36.6903) (layer Edge.Cuts) (width 0.2))
+  (gr_line (start 217.79552 42.621355) (end 171.704 35.687) (layer Edge.Cuts) (width 0.2))
   (gr_line (start 171.53204 135.649242) (end 171.277232 135.787458) (layer Edge.Cuts) (width 0.2))
   (gr_line (start 171.753993 135.466153) (end 171.53204 135.649242) (layer Edge.Cuts) (width 0.2))
@@
   (gr_line (start 172.19308 134.427634) (end 172.162633 134.707736) (layer Edge.Cuts) (width 0.2))
   (gr_line (start 219.70492 44.8564) (end 219.70492 119.6848) (layer Edge.Cuts) (width 0.2))
-  (gr_line (start 81.163697 36.869721) (end 81.342063 36.77297) (layer Edge.Cuts) (width 0.2))
-  (gr_line (start 81.00833 36.997883) (end 81.163697 36.869721) (layer Edge.Cuts) (width 0.2))
-  (gr_line (start 80.880169 37.153249) (end 81.00833 36.997883) (layer Edge.Cuts) (width 0.2))
-  (gr_line (start 80.783417 37.331615) (end 80.880169 37.153249) (layer Edge.Cuts) (width 0.2))
-  (gr_line (start 80.722283 37.528775) (end 80.783417 37.331615) (layer Edge.Cuts) (width 0.2))
-  (gr_line (start 80.7003 37.7444) (end 80.722283 37.528775) (layer Edge.Cuts) (width 0.2))
-  (gr_line (start 81.539222 36.711835) (end 81.7544 36.6903) (layer Edge.Cuts) (width 0.2))
-  (gr_line (start 81.342063 36.77297) (end 81.539222 36.711835) (layer Edge.Cuts) (width 0.2))
-  (gr_line (start 181.0004 36.6903) (end 81.7544 36.6903) (layer Edge.Cuts) (width 0.2))
-  (gr_line (start 80.645 110.617) (end 80.7003 37.7444) (layer Edge.Cuts) (width 0.2))
+  (gr_line (start 81.163697 35.869721) (end 81.342063 35.77297) (layer Edge.Cuts) (width 0.2))
+  (gr_line (start 81.00833 35.997883) (end 81.163697 35.869721) (layer Edge.Cuts) (width 0.2))
+  (gr_line (start 80.880169 36.153249) (end 81.00833 35.997883) (layer Edge.Cuts) (width 0.2))
+  (gr_line (start 80.783417 36.331615) (end 80.880169 36.153249) (layer Edge.Cuts) (width 0.2))
+  (gr_line (start 80.722283 36.528775) (end 80.783417 36.331615) (layer Edge.Cuts) (width 0.2))
+  (gr_line (start 80.7003 36.7444) (end 80.722283 36.528775) (layer Edge.Cuts) (width 0.2))
+  (gr_line (start 81.539222 35.711835) (end 81.7544 35.6903) (layer Edge.Cuts) (width 0.2))
+  (gr_line (start 81.342063 35.77297) (end 81.539222 35.711835) (layer Edge.Cuts) (width 0.2))
+  (gr_line (start 171.704 35.687) (end 81.7544 35.6903) (layer Edge.Cuts) (width 0.2))
+  (gr_line (start 80.645 110.617) (end 80.7003 36.7444) (layer Edge.Cuts) (width 0.2))
   (gr_line (start 81.4197 116.3955) (end 81.9785 117.6655) (layer Edge.Cuts) (width 0.2))
   (gr_line (start 81.153 115.3795) (end 81.4197 116.3955) (layer Edge.Cuts) (width 0.2))
@@
     (polygon
       (pts
-        (xy 72.6821 37.104) (xy 219.9 37) (xy 219.9 121) (xy 173.9 121) (xy 173.9 136)
+        (xy 72.54265 35.2056) (xy 219.76055 35.1016) (xy 219.9 121) (xy 173.9 121) (xy 173.9 136)
         (xy 111.9 136) (xy 97.9 144) (xy 84.074 119.888) (xy 72.6821 103.104)
       )
@@
     (polygon
       (pts
-        (xy 73.025 36.3293) (xy 219.9 37) (xy 219.9 121) (xy 173.9 121) (xy 173.9 136)
+        (xy 72.7649 34.81825) (xy 219.6399 35.48895) (xy 219.9 121) (xy 173.9 121) (xy 173.9 136)
         (xy 111.9 136) (xy 97.9 144) (xy 84.201 119.888) (xy 73.025 102.3293)
       )
