File: Plate/Glow/MX/FR4_Top_Plate.kicad_pcb (KiCad board)
At the start: 2 copper layers, 139.1 x 106.7 mm, 35 parts, among them SW1 SW_PUSH, SW10 SW_PUSH, SW11 SW_PUSH, SW12 SW_PUSH, SW13 SW_PUSH, SW14 SW_PUSH, SW15 SW_PUSH, SW16 SW_PUSH, SW18 SW_PUSH, SW19 SW_PUSH, SW2 SW_PUSH, SW20 SW_PUSH, SW21 SW_PUSH, SW22 SW_PUSH, SW23 SW_PUSH, SW24 SW_PUSH, SW25 SW_PUSH, SW26 SW_PUSH, SW27 SW_PUSH, SW28 SW_PUSH, SW29 SW_PUSH, SW3 SW_PUSH, SW30 Rotary_Encoder_Switch, SW4 SW_PUSH, SW5 SW_PUSH, SW6 SW_PUSH, SW7 SW_PUSH, SW8 SW_PUSH, SW9 SW_PUSH

Commit message: Updated Plates
Parts:
- removed the SW11 at (190.6, 90.5)
- added SW17: SW_PUSH, Keyboard Library:Cherry_MX_Plate_Hole_Placeholder, F.Cu at (190.6, 90.5)
- moved SW30 1.00 mm to (91.6, 54.6)
Other:
- board size 139.1 x 106.7 mm -> 139.1 x 107.7 mm
- board text removed: "Split 58 HS-RGB"

Commit message: Adjusted plate
Parts:
- SW1, SW10, SW11, SW12, SW13, SW14, SW15, SW16, SW17, SW18, SW19, SW2, SW20, SW21, SW22, SW23, SW24, SW25, SW26, SW27, SW28, SW29, SW3, SW4, SW5, SW6, SW7, SW8, SW9: footprint Keyboard Library:Cherry_MX_Plate_Hole_Placeholder -> Keyboard Library:Cherry_MX_Plate_Hole_Breakoff
- SW30: footprint Keyboard Library:RotaryEncoder_PlateHole_Placeholder -> Keyboard Library:RotaryEncoder_PlateHole_Breakoff
