File: Wireless/PCB/Lotus58_Wireless.sch (KiCad schematic (older format))
At the start: 69 parts, among them SW1 SW_PUSH, SW10 SW_PUSH, SW11 SW_PUSH, SW12 SW_PUSH, SW13 SW_PUSH, SW14 SW_PUSH, SW15 SW_PUSH, SW16 SW_PUSH, SW17 SW_PUSH, SW18 SW_PUSH, SW19 SW_PUSH, SW2 SW_PUSH, SW20 SW_PUSH, SW21 SW_PUSH, SW22 SW_PUSH, SW23 SW_PUSH, SW24 SW_PUSH, SW25 SW_PUSH, SW26 SW_PUSH, SW27 SW_PUSH, SW28 SW_PUSH, SW29 SW_PUSH, SW3 SW_PUSH, SW30 Rotary_Encoder_Switch, SW4 SW_PUSH, SW5 SW_PUSH, SW6 SW_PUSH, SW7 SW_PUSH, SW8 SW_PUSH, SW9 SW_PUSH

Commit message: RGB midmount footprints
Fixed mirror image pinout
Parts:
- removed D30: 1N4148W, Diode_SMD:D_SOD-123, symbol Device:D
- removed SW30: Rotary_Encoder_Switch, Keebio-Parts:RotaryEncoder_EC11-no-legs, symbol Device:Rotary_Encoder_Switch
- added BT1, BT2: Battery_Cell, Keyboard Library:BAT_BK-888, symbol Device:Battery_Cell
- added D30: BAT60A, Diode_SMD:D_SOD-323, symbol Diode:BAT60A
- added J1: Conn_01x04, Connector_PinHeader_2.54mm:PinHeader_1x04_P2.54mm_Vertical, symbol Connector_Generic:Conn_01x04
- added JP1: Jumper_3_Open, Jumper:SolderJumper-3_P1.3mm_Open_RoundedPad1.0x1.5mm, symbol Jumper:Jumper_3_Open
- added Q1: SI2393DS-T1-GE3, SOT95P237X112-3N, symbol SamacSys_Parts:SI2393DS-T1-GE3
- added R1: 3k3, Resistor_SMD:R_0603_1608Metric_Pad0.98x0.95mm_HandSolder, symbol Device:R
- added U1: Core51822B, Keyboard Library:Core51822(B)_y14015, symbol Keyboard_Library:Core51822B
- added U2: MCP1802x-xx02xOT, Package_TO_SOT_SMD:SOT-23-5, symbol Regulator_Linear:MCP1802x-xx02xOT
- C1, C2: value C_Small -> 1uF; footprint Keyboard Library:RESISTOR_Reversible -> Capacitor_SMD:C_0603_1608Metric_Pad1.05x0.95mm_HandSolder
- SW1, SW10, SW11, SW12, SW13, SW14, SW15, SW16, SW17, SW18, SW19, SW2, SW20, SW21, SW22, SW23, SW24, SW25, SW26, SW27, SW28, SW29, SW3, SW4, SW5, SW6, SW7, SW8, SW9: footprint keyswitches:Kailh_socket_MX_reversible_RGB -> keyswitches:Kaih_socket_MX_Choc_V1&V2_reversible
- TH3, TH4, TH5, TH6, TH7: footprint MountingHole:MountingHole_2.7mm_M2.5 -> MountingHole:MountingHole_3.2mm_M3
Connections:
- net labels added: +3V3, +BATT, POWER, SWCLK, SWDIO, VPP
- net labels removed: A, Alt, B, DATA, Enc0, Enc1, LED, MISO, MOSI, RESET, RST, SCK, SCL, SDA
- wire segments 117 -> 136
- no-connect marks 1 -> 19
Other:
- moved on the sheet: JP12, JP13, TH3, TH4, TH5, TH6, TH7
