File: Glow/PCB/MX/Lotus58_Glow.sch (KiCad schematic (older format))
At the start: 122 parts, among them J1 AudioJack4, P4 OLED, SW1 SW_PUSH, SW10 SW_PUSH, SW11 SW_PUSH, SW12 SW_PUSH, SW13 SW_PUSH, SW14 SW_PUSH, SW15 SW_PUSH, SW16 SW_PUSH, SW17 SW_PUSH, SW18 SW_PUSH, SW19 SW_PUSH, SW2 SW_PUSH, SW20 SW_PUSH, SW21 SW_PUSH, SW22 SW_PUSH, SW23 SW_PUSH, SW24 SW_PUSH, SW25 SW_PUSH, SW26 SW_PUSH, SW27 SW_PUSH, SW28 SW_PUSH, SW29 SW_PUSH, SW3 SW_PUSH, SW30 Rotary_Encoder_Switch, SW31 Rotary_Encoder_Switch, SW4 SW_PUSH, SW5 SW_PUSH, SW6 SW_PUSH, SW7 SW_PUSH, SW8 SW_PUSH, SW9 SW_PUSH, U1 ProMicro

Commit message: RGB midmount footprints
Fixed mirror image pinout
Parts:
- L1, L10, L11, L12, L13, L14, L15, L16, L17, L18, L19, L2, L20, L21, L22, L23, L24, L25, L26, L27, L28, L29, L3, L30, L31, L32, L33, L34, L35, L4, L5, L6, L7, L8, L9: symbol LED:SK6812MINI -> Keyboard_Library:SK6812MINI
Connections:
- net GND: now also L1.1 (VSS), L10.1 (VSS), L11.1 (VSS), L12.1 (VSS), L13.1 (VSS), L14.1 (VSS), L15.1 (VSS), L16.1 (VSS), L17.1 (VSS), L18.1 (VSS), L19.1 (VSS), L2.1 (VSS), L20.1 (VSS), L21.1 (VSS), L22.1 (VSS), L23.1 (VSS), L24.1 (VSS), L25.1 (VSS), L26.1 (VSS), L27.1 (VSS), L28.1 (VSS), L29.1 (VSS), L3.1 (VSS), L30.1 (VSS), L31.1 (VSS), L32.1 (VSS), L33.1 (VSS), L34.1 (VSS), L35.1 (VSS), L4.1 (VSS), L5.1 (VSS), L6.1 (VSS), L7.1 (VSS), L8.1 (VSS), L9.1 (VSS); no longer L1.2 (VSS), L10.2 (VSS), L11.2 (VSS), L12.2 (VSS), L13.2 (VSS), L14.2 (VSS), L15.2 (VSS), L16.2 (VSS), L17.2 (VSS), L18.2 (VSS), L19.2 (VSS), L2.2 (VSS), L20.2 (VSS), L21.2 (VSS), L22.2 (VSS), L23.2 (VSS), L24.2 (VSS), L25.2 (VSS), L26.2 (VSS), L27.2 (VSS), L28.2 (VSS), L29.2 (VSS), L3.2 (VSS), L30.2 (VSS), L31.2 (VSS), L32.2 (VSS), L33.2 (VSS), L34.2 (VSS), L35.2 (VSS), L4.2 (VSS), L5.2 (VSS), L6.2 (VSS), L7.2 (VSS), L8.2 (VSS), L9.2 (VSS)
- net LED: now also L1.2 (DIN); no longer L1.3 (DIN)
- net VCC: now also L1.3 (VDD), L10.3 (VDD), L11.3 (VDD), L12.3 (VDD), L13.3 (VDD), L14.3 (VDD), L15.3 (VDD), L16.3 (VDD), L17.3 (VDD), L18.3 (VDD), L19.3 (VDD), L2.3 (VDD), L20.3 (VDD), L21.3 (VDD), L22.3 (VDD), L23.3 (VDD), L24.3 (VDD), L25.3 (VDD), L26.3 (VDD), L27.3 (VDD), L28.3 (VDD), L29.3 (VDD), L3.3 (VDD), L30.3 (VDD), L31.3 (VDD), L32.3 (VDD), L33.3 (VDD), L34.3 (VDD), L35.3 (VDD), L4.3 (VDD), L5.3 (VDD), L6.3 (VDD), L7.3 (VDD), L8.3 (VDD), L9.3 (VDD); no longer L1.4 (VDD), L10.4 (VDD), L11.4 (VDD), L12.4 (VDD), L13.4 (VDD), L14.4 (VDD), L15.4 (VDD), L16.4 (VDD), L17.4 (VDD), L18.4 (VDD), L19.4 (VDD), L2.4 (VDD), L20.4 (VDD), L21.4 (VDD), L22.4 (VDD), L23.4 (VDD), L24.4 (VDD), L25.4 (VDD), L26.4 (VDD), L27.4 (VDD), L28.4 (VDD), L29.4 (VDD), L3.4 (VDD), L30.4 (VDD), L31.4 (VDD), L32.4 (VDD), L33.4 (VDD), L34.4 (VDD), L35.4 (VDD), L4.4 (VDD), L5.4 (VDD), L6.4 (VDD), L7.4 (VDD), L8.4 (VDD), L9.4 (VDD)
- new net: L1.4 (DOUT), L35.2 (DIN)
- new net: L2.2 (DIN), L35.4 (DOUT)
- new net: L2.4 (DOUT), L3.2 (DIN)
- new net: L3.4 (DOUT), L34.2 (DIN)
- new net: L34.4 (DOUT), L4.2 (DIN)
- new net: L4.4 (DOUT), L5.2 (DIN)
- new net: L33.2 (DIN), L5.4 (DOUT)
- new net: L33.4 (DOUT), L6.2 (DIN)
- new net: L12.2 (DIN), L6.4 (DOUT)
- new net: L7.2 (DIN), L8.4 (DOUT)
- new net: L13.2 (DIN), L7.4 (DOUT)
- new net: L8.2 (DIN), L9.4 (DOUT)
- new net: L10.4 (DOUT), L9.2 (DIN)
- new net: L10.2 (DIN), L11.4 (DOUT)
- new net: L11.2 (DIN), L12.4 (DOUT)
- new net: L13.4 (DOUT), L14.2 (DIN)
- new net: L14.4 (DOUT), L15.2 (DIN)
- new net: L15.4 (DOUT), L16.2 (DIN)
- new net: L16.4 (DOUT), L17.2 (DIN)
- new net: L17.4 (DOUT), L18.2 (DIN)
- new net: L18.4 (DOUT), L24.2 (DIN)
- new net: L19.2 (DIN), L20.4 (DOUT)
- new net: L19.4 (DOUT), L32.2 (DIN)
- new net: L20.2 (DIN), L21.4 (DOUT)
- new net: L21.2 (DIN), L22.4 (DOUT)
- new net: L22.2 (DIN), L23.4 (DOUT)
- new net: L23.2 (DIN), L30.4 (DOUT)
- new net: L24.4 (DOUT), L30.2 (DIN)
- new net: L25.2 (DIN), L32.4 (DOUT)
- new net: L25.4 (DOUT), L26.2 (DIN)
- new net: L26.4 (DOUT), L27.2 (DIN)
- new net: L27.4 (DOUT), L28.2 (DIN)
- new net: L28.4 (DOUT), L31.2 (DIN)
- new net: L29.2 (DIN), L31.4 (DOUT)
Changed lines of the file:
@@
 	3350 9750 3550 9750
 $Comp
-L LED:SK6812MINI L28
+L Keyboard_Library:SK6812MINI L28
 U 1 1 5D44C2D1
 P 4650 9750
@@
 $EndComp
 $Comp
-L LED:SK6812MINI L27
+L Keyboard_Library:SK6812MINI L27
 U 1 1 5D44C2CB
 P 3850 9750
@@
 	2550 9750 2750 9750
 $Comp
-L LED:SK6812MINI L26
+L Keyboard_Library:SK6812MINI L26
 U 1 1 5D44C2C0
 P 3050 9750
@@
 $EndComp
 $Comp
-L LED:SK6812MINI L25
+L Keyboard_Library:SK6812MINI L25
 U 1 1 5D44C2AB
 P 2250 9750
@@
 	3350 9050 3550 9050
 $Comp
-L LED:SK6812MINI L24
+L Keyboard_Library:SK6812MINI L24
 U 1 1 5D3B3CCB
 P 8000 9050
@@
 $EndComp
 $Comp
-L LED:SK6812MINI L23
+L Keyboard_Library:SK6812MINI L23
 U 1 1 5D3B3CC5
 P 6250 9050
@@
 $EndComp
 $Comp
-L LED:SK6812MINI L22
+L Keyboard_Library:SK6812MINI L22
 U 1 1 5D3B3CBF
 P 5450 9050
@@
 $EndComp
 $Comp
-L LED:SK6812MINI L21
+L Keyboard_Library:SK6812MINI L21
 U 1 1 5D3B3CB9
 P 4650 9050
@@
 	2550 9050 2750 9050
 $Comp
-L LED:SK6812MINI L20
+L Keyboard_Library:SK6812MINI L20
 U 1 1 5D3B3CB0
 P 3850 9050
@@
 $EndComp
 $Comp
-L LED:SK6812MINI L19
+L Keyboard_Library:SK6812MINI L19
 U 1 1 5D3B3C9E
 P 3050 9050
@@
 	3350 8350 3550 8350
 $Comp
-L LED:SK6812MINI L18
+L Keyboard_Library:SK6812MINI L18
 U 1 1 5D3B3C84
 P 6250 8350
@@
 $EndComp
 $Comp
-L LED:SK6812MINI L17
+L Keyboard_Library:SK6812MINI L17
 U 1 1 5D3B3C7E
 P 5450 8350
@@
 $EndComp
 $Comp
-L LED:SK6812MINI L16
+L Keyboard_Library:SK6812MINI L16
 U 1 1 5D3B3C78
 P 4650 8350
@@
 $EndComp
 $Comp
-L LED:SK6812MINI L15
+L Keyboard_Library:SK6812MINI L15
 U 1 1 5D3B3C72
 P 3850 8350
@@
 	2550 8350 2750 8350
 $Comp
-L LED:SK6812MINI L14
+L Keyboard_Library:SK6812MINI L14
 U 1 1 5D3B3C67
 P 3050 8350
@@
 $EndComp
 $Comp
-L LED:SK6812MINI L13
+L Keyboard_Library:SK6812MINI L13
 U 1 1 5D3B3C52
 P 2250 8350
@@
 	3350 7650 3550 7650
 $Comp
-L LED:SK6812MINI L12
+L Keyboard_Library:SK6812MINI L12
 U 1 1 5D36810E
 P 6250 7650
@@
 $EndComp
 $Comp
-L LED:SK6812MINI L11
+L Keyboard_Library:SK6812MINI L11
 U 1 1 5D368108
 P 5450 7650
@@
 $EndComp
 $Comp
-L LED:SK6812MINI L10
+L Keyboard_Library:SK6812MINI L10
 U 1 1 5D368102
 P 4650 7650
@@
 $EndComp
 $Comp
-L LED:SK6812MINI L9
+L Keyboard_Library:SK6812MINI L9
 U 1 1 5D3680FC
 P 3850 7650
@@
 	2550 7650 2750 7650
 $Comp
-L LED:SK6812MINI L8
+L Keyboard_Library:SK6812MINI L8
 U 1 1 5D3680F1
 P 3050 7650
@@
 	3050 6650 3850 6650
 $Comp
-L LED:SK6812MINI L6
+L Keyboard_Library:SK6812MINI L6
 U 1 1 5D33FFE4
 P 8850 6950
@@
 $EndComp
 $Comp
-L LED:SK6812MINI L5
+L Keyboard_Library:SK6812MINI L5
 U 1 1 5D33BE08
 P 7100 6950
@@
 $EndComp
 $Comp
-L LED:SK6812MINI L4
+L Keyboard_Library:SK6812MINI L4
 U 1 1 5D3368F0
 P 6250 6950
@@
 $EndComp
 $Comp
-L LED:SK6812MINI L3
+L Keyboard_Library:SK6812MINI L3
 U 1 1 5D3339D0
 P 4650 6950
@@
 	2550 6950 2750 6950
 $Comp
-L LED:SK6812MINI L2
+L Keyboard_Library:SK6812MINI L2
 U 1 1 5D319DBE
 P 3850 6950
@@
 $EndComp
 $Comp
-L LED:SK6812MINI L1
+L Keyboard_Library:SK6812MINI L1
 U 1 1 5D2E8536
 P 2250 6950
@@
 $EndComp
 $Comp
-L LED:SK6812MINI L29
+L Keyboard_Library:SK6812MINI L29
 U 1 1 5D5C8664
 P 6250 9750
@@
 	2700 3400 2700 3250
 $Comp
-L LED:SK6812MINI L30
+L Keyboard_Library:SK6812MINI L30
 U 1 1 5FBC8279
 P 7150 9050
@@
 $EndComp
 $Comp
-L LED:SK6812MINI L31
+L Keyboard_Library:SK6812MINI L31
 U 1 1 5FBC951D
 P 5450 9750
@@
 $EndComp
 $Comp
-L LED:SK6812MINI L32
+L Keyboard_Library:SK6812MINI L32
 U 1 1 5FBC9BCE
 P 2250 9050
@@
 $EndComp
 $Comp
-L LED:SK6812MINI L35
+L Keyboard_Library:SK6812MINI L35
 U 1 1 5FBCA361
 P 3050 6950
@@
 $EndComp
 $Comp
-L LED:SK6812MINI L7
+L Keyboard_Library:SK6812MINI L7
 U 1 1 5D3680DC
 P 2250 7650
@@
 	7700 6950 7400 6950
 $Comp
-L LED:SK6812MINI L33
+L Keyboard_Library:SK6812MINI L33
 U 1 1 5FBCBCC4
 P 8000 6950
@@
 $EndComp
 $Comp
-L LED:SK6812MINI L34
+L Keyboard_Library:SK6812MINI L34
 U 1 1 5FBCB693
 P 5450 6950

Commit message: Component values/BOM added
Parts:
- C1, C2: value C_Small -> 100nF
- D1, D10, D11, D12, D13, D14, D15, D16, D17, D18, D19, D2, D20, D21, D22, D23, D24, D25, D26, D27, D28, D29, D3, D30, D4, D5, D6, D7, D8, D9: value D -> 1N4148/1N4148W
- J1: value AudioJack4 -> PJ-320A
- JP12: value LH -> Jumper_NO_Small
- JP13: value RH -> Jumper_NO_Small
- R1, R2: value R -> 4k7
- SW1, SW10, SW11, SW12, SW13, SW14, SW15, SW16, SW17, SW18, SW19, SW2, SW20, SW21, SW22, SW23, SW24, SW25, SW26, SW27, SW28, SW29, SW3, SW4, SW5, SW6, SW7, SW8, SW9: value SW_PUSH -> Kailh hotswap MX socket
