File: PCB/Lotus58_Glow.kicad_pcb (KiCad board)
At the start: 2 copper layers, 139.1 x 107.7 mm, 133 parts, among them J1 PJ-320A, J2 Conn_01x02, P1 OLED, SW1 Kailh hotswap MX socket, SW10 Kailh hotswap MX socket, SW11 Kailh hotswap MX socket, SW12 Kailh hotswap MX socket, SW13 Kailh hotswap MX socket, SW14 Kailh hotswap MX socket, SW15 Kailh hotswap MX socket, SW16 Kailh hotswap MX socket, SW17 Kailh hotswap MX socket, SW18 Kailh hotswap MX socket, SW19 Kailh hotswap MX socket, SW2 Kailh hotswap MX socket, SW20 Kailh hotswap MX socket, SW21 Kailh hotswap MX socket, SW22 Kailh hotswap MX socket, SW23 Kailh hotswap MX socket, SW24 Kailh hotswap MX socket, SW25 Kailh hotswap MX socket, SW26 Kailh hotswap MX socket, SW27 Kailh hotswap MX socket, SW28 Kailh hotswap MX socket, SW29 Kailh hotswap MX socket, SW3 Kailh hotswap MX socket, SW30 Rotary_Encoder_Switch, SW31 Rotary_Encoder_Switch, SW4 Kailh hotswap MX socket, SW5 Kailh hotswap MX socket, SW6 Kailh hotswap MX socket, SW7 Kailh hotswap MX socket, SW8 Kailh hotswap MX socket, SW9 Kailh hotswap MX socket, U1 ProMicro

Commit message: update
Routing:
- net SCL: track 61.1 -> 50.5 mm
- net GND: track 192.1 -> 187.4 mm, vias 92 -> 93
Other:
- board text added: "JLCJLCJLCJLC"

Commit message: updated v1.22
Parts:
- moved JP16 1.70 mm to (101.4, 87.2)
- moved JP3 1.05 mm to (83.8, 72.9)
- moved JP4 1.05 mm to (83.8, 72.9)
- moved C7 0.95 mm to (142.8, 91.4)
Routing:
- net SCL: track 50.5 -> 65.5 mm, vias 2 -> 3
- net RGB_GLOW: track 27.5 -> 29.4 mm
- net LED: track 67.7 -> 66.3 mm
- net RGB_KEY: track 49.5 -> 48.1 mm
- net A: track 83.0 -> 84.1 mm
- net GND: vias 93 -> 92
- net (no net): vias 0 -> 1
Other:
- board text added: "Capactitors C3 to C11 are optional, and can be left unused."
- board text added: "D30 is optional, and only needed if the encoder is placed in the top position."
- board text added: "Diodes and RGB's MUST be placed in the correct direction to function."
- board text added: "Do NOT solder TRRS if building a wireless keyboard"
- board text added: "LEFT HAND"
- board text added: "Markus Knutsson 2021 - https://github.com/TweetyDaBird - Licensed under CERN-OHL-S v2+"
- board text added: "Optional switch and battery connection for wireless build."
- board text added: "Per key RGB's are placed face down, with the notched corner at the VISIBLE marking as they are soldered."
- board text added: "Place Encoder on TOP of PCB."
- board text added: "Place ProMicro or socket in markings with component side against PCB"
- board text added: "Place stripe of diode at the line/side where arrow is pointing."
- board text added: "RIGHT HAND"
- board text added: "Resistors and capacitors can be placed in either direction."
- board text added: "The COMPONENT side of the PCB is the BACK side for that hand."
- board text added: "Underglow RGB's are placed with the visible marking matching the notch on its face."
- board text added: "Warning: Close ONLY one RGB connection!"
- board text added: "v1.22"
- board text removed: "Fact: Resistors (Rx) and capacitors (Cx) can be placed in either direction."
- board text removed: "Fact: The COMPONENT side of the PCB is the BACK side for that hand."
- board text removed: "HAND"
- board text removed: "Markus Knutsson 2020 - https://github.com/TweetyDaBird - Licensed under CERN-OHL-S v2+"
- board text removed: "Note: Capactitors C3 to C11 are optional, and do not need to be soldered normally."
- board text removed: "Note: Diodes and RGB's are directional and MUST be placed correctly to function."
- board text removed: "Note: Place stripe of diode at the line/side where arrow is pointing."
- board text removed: "Note: SK6812mini RGB LED's (Glow) are placed with the visible marking matching the notch on its face."
- board text removed: "Note: SK6812mini-E RGB LED's are placed on top of the PCB face down, with the notched corner at the VISIBLE marking as they are soldered."
- board text removed: "Note: The diode D30 is optional, and only needed if the encoder is placed in the top position."
- board text removed: "Optional battery switch and battery connection for wireless build."
- board text removed: "Place ProMicro in markings with component side against PCB"
- board text removed: "Warning: Close ONLY one connection, from middle pad to either GLOW or KEY"
- board text removed: "Warning: Do NOT solder TRRS if building a wireless keyboard"
- board text removed: "Warning: The RGB's are placed in different direction on different rows."
- board text removed: "v1.21"
