File: PCB/Lotus58_Glow.kicad_pcb (KiCad board)
At the start: 2 copper layers, 139.1 x 107.7 mm, 133 parts, among them J1 PJ-320A, J2 Conn_01x02, P1 OLED, SW1 Kailh hotswap MX socket, SW10 Kailh hotswap MX socket, SW11 Kailh hotswap MX socket, SW12 Kailh hotswap MX socket, SW13 Kailh hotswap MX socket, SW14 Kailh hotswap MX socket, SW15 Kailh hotswap MX socket, SW16 Kailh hotswap MX socket, SW17 Kailh hotswap MX socket, SW18 Kailh hotswap MX socket, SW19 Kailh hotswap MX socket, SW2 Kailh hotswap MX socket, SW20 Kailh hotswap MX socket, SW21 Kailh hotswap MX socket, SW22 Kailh hotswap MX socket, SW23 Kailh hotswap MX socket, SW24 Kailh hotswap MX socket, SW25 Kailh hotswap MX socket, SW26 Kailh hotswap MX socket, SW27 Kailh hotswap MX socket, SW28 Kailh hotswap MX socket, SW29 Kailh hotswap MX socket, SW3 Kailh hotswap MX socket, SW30 Rotary_Encoder_Switch, SW31 Rotary_Encoder_Switch, SW4 Kailh hotswap MX socket, SW5 Kailh hotswap MX socket, SW6 Kailh hotswap MX socket, SW7 Kailh hotswap MX socket, SW8 Kailh hotswap MX socket, SW9 Kailh hotswap MX socket, U1 ProMicro

Commit message: v1.23
Parts:
- R1, R2: footprint Resistor_THT:R_Axial_DIN0204_L3.6mm_D1.6mm_P5.08mm_Horizontal -> Resistor_THT:R_Axial_DIN0207_L6.3mm_D2.5mm_P7.62mm_Horizontal
- moved R1 8.25 mm to (99.7, 79.5), turned to 90 degrees
- moved R2 4.62 mm to (102.4, 79.5), turned to 90 degrees
- moved JP16 2.49 mm to (101.9, 89.7)
- moved JP15 0.48 mm to (101.7, 98.3)
Routing:
- net RGB_KEY: track 48.1 -> 50.8 mm
- net LED: track 66.3 -> 69.0 mm
- net VCC: track 889.3 -> 886.8 mm
- net RGB_GLOW: track 29.4 -> 27.4 mm
- net col1: track 246.9 -> 247.8 mm
- net row2: track 160.1 -> 159.2 mm
- net SDA: track 57.4 -> 56.6 mm
- net row4: track 160.0 -> 159.4 mm
- net SCL: track 65.5 -> 65.0 mm
Other:
- board text added: "v1.23"
- board text removed: "v1.22"
