File: test/Lotus58_Glow.kicad_pcb (KiCad board)
At the start: 2 copper layers, 139.1 x 107.7 mm, 133 parts, among them J1 PJ-320A, J2 Conn_01x02, P1 OLED, SW1 Kailh hotswap MX socket, SW10 Kailh hotswap MX socket, SW11 Kailh hotswap MX socket, SW12 Kailh hotswap MX socket, SW13 Kailh hotswap MX socket, SW14 Kailh hotswap MX socket, SW15 Kailh hotswap MX socket, SW16 Kailh hotswap MX socket, SW17 Kailh hotswap MX socket, SW18 Kailh hotswap MX socket, SW19 Kailh hotswap MX socket, SW2 Kailh hotswap MX socket, SW20 Kailh hotswap MX socket, SW21 Kailh hotswap MX socket, SW22 Kailh hotswap MX socket, SW23 Kailh hotswap MX socket, SW24 Kailh hotswap MX socket, SW25 Kailh hotswap MX socket, SW26 Kailh hotswap MX socket, SW27 Kailh hotswap MX socket, SW28 Kailh hotswap MX socket, SW29 Kailh hotswap MX socket, SW3 Kailh hotswap MX socket, SW30 Rotary_Encoder_Switch, SW31 Rotary_Encoder_Switch, SW4 Kailh hotswap MX socket, SW5 Kailh hotswap MX socket, SW6 Kailh hotswap MX socket, SW7 Kailh hotswap MX socket, SW8 Kailh hotswap MX socket, SW9 Kailh hotswap MX socket, U1 ProMicro

Commit message: updated v1.22
Parts:
- added JP13: Jumper_NO_Small, Keyboard Library:Jumper_Mini, F.Cu at (100.5, 103.4)
- added JP14: Jumper_NO_Small, Keyboard Library:Jumper_Mini, F.Cu at (100.4, 100.9)
- added JP17: Jumper_NO_Small, Keyboard Library:Jumper_Mini, F.Cu at (100.4, 98.4)
- added JP18: Jumper_NO_Small, Keyboard Library:Jumper_Mini, F.Cu at (100.4, 93.3)
- added JP19: Jumper_NO_Small, Keyboard Library:Jumper_Mini, B.Cu at (100.4, 93.3)
- added JP20: Jumper_NO_Small, Keyboard Library:Jumper_Mini, B.Cu at (100.4, 98.4)
- added JP21: Jumper_NO_Small, Keyboard Library:Jumper_Mini, B.Cu at (100.4, 100.9)
- added JP22: Jumper_NO_Small, Keyboard Library:Jumper_Mini, B.Cu at (100.5, 103.4)
- added TRA1: trackball, Keyboard Library:trackball, F.Cu at (90.5, 98.3)
- moved D25 23.6 mm to (89.0, 111.8)
- moved JP15 13.0 mm to (102.5, 84.8), turned to 0 degrees
- moved JP16 5.88 mm to (102.4, 81.4)
Routing:
- net Net-(LED19-Pad2): track 27.6 -> 47.8 mm, vias 2 -> 3
- net Alt: track 16.5 -> 33.3 mm
- net RGB_LINK: track 97.9 -> 111.1 mm
- net (no net): track 0.00 -> 6.76 mm
- net LED: track 66.3 -> 60.0 mm
- net RGB_KEY: track 48.1 -> 41.8 mm
- net RGB_GLOW: track 29.4 -> 34.6 mm
- net Net-(JP17-Pad1): track 0.00 -> 3.21 mm
- net Net-(JP18-Pad1): track 0.00 -> 3.21 mm
- net Net-(JP14-Pad1): track 0.00 -> 3.21 mm
- net Net-(JP13-Pad1): track 0.00 -> 3.19 mm
- net row3: track 172.4 -> 169.3 mm, vias 3 -> 2
- net VCC: track 889.3 -> 892.2 mm
- net Net-(LED30-Pad1): track 76.4 -> 74.4 mm, vias 4 -> 5
- net Net-(LED25-Pad2): track 33.5 -> 32.1 mm
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